File: Base/Schematic/DOUT.kicad_sch (KiCad schematic)
At the start: 12 parts, among them U3 BTS5200-4EKA

Commit message: [Base 회로도 업데이트] - DOUT 출력을 4개에서 8개로 늘림
Parts:
- renumbered C16 to C17, R16 to R25, R23 to R32, R24 to R33, U3 to U4
Changed lines of the file:
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@@
 		(dnp no)
 		(fields_autoplaced yes)
-		(property "Reference" "R23"
+		(property "Reference" "R32"
 			(at 129.54 104.648 0)
 			(do_not_autoplace yes)
@@
 		)
 		(instances
-			(project ""
-				(path "/0d177ca6-e392-45a0-9514-d370436392ef/caced042-0264-4901-a3a6-78acc82068a3"
-					(reference "R23")
+			(project "Open-PLC-Project"
+				(path "/0d177ca6-e392-45a0-9514-d370436392ef/35842953-03b1-4d1a-a0b9-e32cdca1a04c"
+					(reference "R32")
 					(unit 1)
 				)
@@
 		(instances
 			(project "Open-PLC-Project"
+				(path "/0d177ca6-e392-45a0-9514-d370436392ef/35842953-03b1-4d1a-a0b9-e32cdca1a04c"
+					(reference "R31")
+					(unit 1)
+				)
 				(path "/0d177ca6-e392-45a0-9514-d370436392ef/caced042-0264-4901-a3a6-78acc82068a3"
 					(reference "R22")
@@
 		(instances
 			(project "Open-PLC-Project"
+				(path "/0d177ca6-e392-45a0-9514-d370436392ef/35842953-03b1-4d1a-a0b9-e32cdca1a04c"
+					(reference "#PWR034")
+					(unit 1)
+				)
 				(path "/0d177ca6-e392-45a0-9514-d370436392ef/caced042-0264-4901-a3a6-78acc82068a3"
 					(reference "#PWR013")
@@
 		(instances
 			(project "Open-PLC-Project"
+				(path "/0d177ca6-e392-45a0-9514-d370436392ef/35842953-03b1-4d1a-a0b9-e32cdca1a04c"
+					(reference "R29")
+					(unit 1)
+				)
 				(path "/0d177ca6-e392-45a0-9514-d370436392ef/caced042-0264-4901-a3a6-78acc82068a3"
 					(reference "R20")
@@
 		(instances
 			(project "Open-PLC-Project"
+				(path "/0d177ca6-e392-45a0-9514-d370436392ef/35842953-03b1-4d1a-a0b9-e32cdca1a04c"
+					(reference "C39")
+					(unit 1)
+				)
 				(path "/0d177ca6-e392-45a0-9514-d370436392ef/caced042-0264-4901-a3a6-78acc82068a3"
 					(reference "C7")
@@
 		(instances
 			(project "Open-PLC-Project"
+				(path "/0d177ca6-e392-45a0-9514-d370436392ef/35842953-03b1-4d1a-a0b9-e32cdca1a04c"
+					(reference "R27")
+					(unit 1)
+				)
 				(path "/0d177ca6-e392-45a0-9514-d370436392ef/caced042-0264-4901-a3a6-78acc82068a3"
 					(reference "R18")
@@
 		(dnp no)
 		(fields_autoplaced yes)
-		(property "Reference" "#PWR016"
+		(property "Reference" "#PWR029"
 			(at 123.19 119.38 0)
 			(effects
@@
 		)
 		(instances
-			(project ""
-				(path "/0d177ca6-e392-45a0-9514-d370436392ef/caced042-0264-4901-a3a6-78acc82068a3"
-					(reference "#PWR016")
+			(project "Open-PLC-Project"
+				(path "/0d177ca6-e392-45a0-9514-d370436392ef/35842953-03b1-4d1a-a0b9-e32cdca1a04c"
+					(reference "#PWR029")
 					(unit 1)
 				)
@@
 		(instances
 			(project "Open-PLC-Project"
+				(path "/0d177ca6-e392-45a0-9514-d370436392ef/35842953-03b1-4d1a-a0b9-e32cdca1a04c"
+					(reference "R30")
+					(unit 1)
+				)
 				(path "/0d177ca6-e392-45a0-9514-d370436392ef/caced042-0264-4901-a3a6-78acc82068a3"
 					(reference "R21")
@@
 		(instances
 			(project "Open-PLC-Project"
+				(path "/0d177ca6-e392-45a0-9514-d370436392ef/35842953-03b1-4d1a-a0b9-e32cdca1a04c"
+					(reference "#PWR066")
+					(unit 1)
+				)
 				(path "/0d177ca6-e392-45a0-9514-d370436392ef/caced042-0264-4901-a3a6-78acc82068a3"
 					(reference "#PWR028")
@@
 		(instances
 			(project "Open-PLC-Project"
+				(path "/0d177ca6-e392-45a0-9514-d370436392ef/35842953-03b1-4d1a-a0b9-e32cdca1a04c"
+					(reference "#PWR033")
+					(unit 1)
+				)
 				(path "/0d177ca6-e392-45a0-9514-d370436392ef/caced042-0264-4901-a3a6-78acc82068a3"
 					(reference "#PWR012")
@@
 		(on_board yes)
 		(dnp no)
-		(property "Reference" "R16"
+		(property "Reference" "R25"
 			(at 134.62 82.55 0)
 			(do_not_autoplace yes)
@@
 		)
 		(instances
-			(project ""
-				(path "/0d177ca6-e392-45a0-9514-d370436392ef/caced042-0264-4901-a3a6-78acc82068a3"
-					(reference "R16")
+			(project "Open-PLC-Project"
+				(path "/0d177ca6-e392-45a0-9514-d370436392ef/35842953-03b1-4d1a-a0b9-e32cdca1a04c"
+					(reference "R25")
 					(unit 1)
 				)
@@
 		(instances
 			(project "Open-PLC-Project"
+				(path "/0d177ca6-e392-45a0-9514-d370436392ef/35842953-03b1-4d1a-a0b9-e32cdca1a04c"
+					(reference "#PWR032")
+					(unit 1)
+				)
 				(path "/0d177ca6-e392-45a0-9514-d370436392ef/caced042-0264-4901-a3a6-78acc82068a3"
 					(reference "#PWR014")
@@
 		(instances
 			(project "Open-PLC-Project"
+				(path "/0d177ca6-e392-45a0-9514-d370436392ef/35842953-03b1-4d1a-a0b9-e32cdca1a04c"
+					(reference "R28")
+					(unit 1)
+				)
 				(path "/0d177ca6-e392-45a0-9514-d370436392ef/caced042-0264-4901-a3a6-78acc82068a3"
 					(reference "R19")
@@
 		(dnp no)
 		(fields_autoplaced yes)
-		(property "Reference" "R24"
+		(property "Reference" "R33"
 			(at 133.858 113.03 0)
 			(do_not_autoplace yes)
@@
 		)
 		(instances
-			(project ""
-				(path "/0d177ca6-e392-45a0-9514-d370436392ef/caced042-0264-4901-a3a6-78acc82068a3"
-					(reference "R24")
+			(project "Open-PLC-Project"
+				(path "/0d177ca6-e392-45a0-9514-d370436392ef/35842953-03b1-4d1a-a0b9-e32cdca1a04c"
+					(reference "R33")
 					(unit 1)
 				)
@@
 		(instances
 			(project "Open-PLC-Project"
+				(path "/0d177ca6-e392-45a0-9514-d370436392ef/35842953-03b1-4d1a-a0b9-e32cdca1a04c"
+					(reference "R26")
+					(unit 1)
+				)
 				(path "/0d177ca6-e392-45a0-9514-d370436392ef/caced042-0264-4901-a3a6-78acc82068a3"
 					(reference "R17")
@@
 		(dnp no)
 		(fields_autoplaced yes)
-		(property "Reference" "U3"
+		(property "Reference" "U4"
 			(at 146.05 80.01 0)
 			(do_not_autoplace yes)
@@
 		)
 		(instances
-			(project ""
-				(path "/0d177ca6-e392-45a0-9514-d370436392ef/caced042-0264-4901-a3a6-78acc82068a3"
-					(reference "U3")
+			(project "Open-PLC-Project"
+				(path "/0d177ca6-e392-45a0-9514-d370436392ef/35842953-03b1-4d1a-a0b9-e32cdca1a04c"
+					(reference "U4")
 					(unit 1)
 				)
@@
 		(dnp no)
 		(fields_autoplaced yes)
-		(property "Reference" "C16"
+		(property "Reference" "C17"
 			(at 124.46 111.76 0)
 			(do_not_autoplace yes)
@@
 		)
 		(instances
-			(project ""
-				(path "/0d177ca6-e392-45a0-9514-d370436392ef/caced042-0264-4901-a3a6-78acc82068a3"
-					(reference "C16")
+			(project "Open-PLC-Project"
+				(path "/0d177ca6-e392-45a0-9514-d370436392ef/35842953-03b1-4d1a-a0b9-e32cdca1a04c"
+					(reference "C17")
 					(unit 1)
 				)
@@
 		(instances
 			(project "Open-PLC-Project"
+				(path "/0d177ca6-e392-45a0-9514-d370436392ef/35842953-03b1-4d1a-a0b9-e32cdca1a04c"
+					(reference "#PWR067")
+					(unit 1)
+				)
 				(path "/0d177ca6-e392-45a0-9514-d370436392ef/caced042-0264-4901-a3a6-78acc82068a3"
 					(reference "#PWR027")

Commit message: [Base PCB 업데이트] - PCB 외곽선과 볼트 위치 설정
Parts:
- renumbered C17 to C41, C7 to C42, R17 to R26, R18 to R27, R19 to R28, R20 to R29, R21 to R30, R22 to R31, U4 to U11
Changed lines of the file:
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@@
+					(unit 1)
+				)
+				(path "/0d177ca6-e392-45a0-9514-d370436392ef/caced042-0264-4901-a3a6-78acc82068a3"
+					(reference "R23")
 					(unit 1)
 				)
@@
 		(on_board yes)
 		(dnp no)
-		(property "Reference" "R22"
+		(property "Reference" "R31"
 			(at 134.62 100.33 0)
 			(do_not_autoplace yes)
@@
 		(dnp no)
 		(fields_autoplaced yes)
-		(property "Reference" "#PWR013"
+		(property "Reference" "#PWR070"
 			(at 166.37 109.22 0)
 			(effects
@@
 			(project "Open-PLC-Project"
 				(path "/0d177ca6-e392-45a0-9514-d370436392ef/35842953-03b1-4d1a-a0b9-e32cdca1a04c"
-					(reference "#PWR034")
-					(unit 1)
-				)
-				(path "/0d177ca6-e392-45a0-9514-d370436392ef/caced042-0264-4901-a3a6-78acc82068a3"
-					(reference "#PWR013")
+					(reference "#PWR070")
+					(unit 1)
+				)
+				(path "/0d177ca6-e392-45a0-9514-d370436392ef/caced042-0264-4901-a3a6-78acc82068a3"
+					(reference "#PWR064")
 					(unit 1)
 				)
@@
 		(on_board yes)
 		(dnp no)
-		(property "Reference" "R20"
+		(property "Reference" "R29"
 			(at 134.62 95.25 0)
 			(do_not_autoplace yes)
@@
 		(dnp no)
 		(fields_autoplaced yes)
-		(property "Reference" "C7"
+		(property "Reference" "C42"
 			(at 175.26 76.2 0)
 			(do_not_autoplace yes)
@@
 			(project "Open-PLC-Project"
 				(path "/0d177ca6-e392-45a0-9514-d370436392ef/35842953-03b1-4d1a-a0b9-e32cdca1a04c"
-					(reference "C39")
-					(unit 1)
-				)
-				(path "/0d177ca6-e392-45a0-9514-d370436392ef/caced042-0264-4901-a3a6-78acc82068a3"
-					(reference "C7")
+					(reference "C42")
+					(unit 1)
+				)
+				(path "/0d177ca6-e392-45a0-9514-d370436392ef/caced042-0264-4901-a3a6-78acc82068a3"
+					(reference "C40")
 					(unit 1)
 				)
@@
 		(on_board yes)
 		(dnp no)
-		(property "Reference" "R18"
+		(property "Reference" "R27"
 			(at 134.62 87.63 0)
 			(do_not_autoplace yes)
@@
 		(dnp no)
 		(fields_autoplaced yes)
-		(property "Reference" "#PWR029"
+		(property "Reference" "#PWR067"
 			(at 123.19 119.38 0)
 			(effects
@@
 			(project "Open-PLC-Project"
 				(path "/0d177ca6-e392-45a0-9514-d370436392ef/35842953-03b1-4d1a-a0b9-e32cdca1a04c"
-					(reference "#PWR029")
+					(reference "#PWR067")
+					(unit 1)
+				)
+				(path "/0d177ca6-e392-45a0-9514-d370436392ef/caced042-0264-4901-a3a6-78acc82068a3"
+					(reference "#PWR061")
 					(unit 1)
 				)
@@
 		(on_board yes)
 		(dnp no)
-		(property "Reference" "R21"
+		(property "Reference" "R30"
 			(at 134.62 97.79 0)
 			(do_not_autoplace yes)
@@
 		(dnp no)
 		(fields_autoplaced yes)
-		(property "Reference" "#PWR028"
+		(property "Reference" "#PWR071"
 			(at 173.99 71.374 0)
 			(effects
@@
 			(project "Open-PLC-Project"
 				(path "/0d177ca6-e392-45a0-9514-d370436392ef/35842953-03b1-4d1a-a0b9-e32cdca1a04c"
-					(reference "#PWR066")
-					(unit 1)
-				)
-				(path "/0d177ca6-e392-45a0-9514-d370436392ef/caced042-0264-4901-a3a6-78acc82068a3"
-					(reference "#PWR028")
+					(reference "#PWR071")
+					(unit 1)
+				)
+				(path "/0d177ca6-e392-45a0-9514-d370436392ef/caced042-0264-4901-a3a6-78acc82068a3"
+					(reference "#PWR065")
 					(unit 1)
 				)
@@
 		(dnp no)
 		(fields_autoplaced yes)
-		(property "Reference" "#PWR012"
+		(property "Reference" "#PWR069"
 			(at 166.37 78.994 0)
 			(effects
@@
 			(project "Open-PLC-Project"
 				(path "/0d177ca6-e392-45a0-9514-d370436392ef/35842953-03b1-4d1a-a0b9-e32cdca1a04c"
-					(reference "#PWR033")
-					(unit 1)
-				)
-				(path "/0d177ca6-e392-45a0-9514-d370436392ef/caced042-0264-4901-a3a6-78acc82068a3"
-					(reference "#PWR012")
+					(reference "#PWR069")
+					(unit 1)
+				)
+				(path "/0d177ca6-e392-45a0-9514-d370436392ef/caced042-0264-4901-a3a6-78acc82068a3"
+					(reference "#PWR063")
 					(unit 1)
 				)
@@
 					(unit 1)
 				)
+				(path "/0d177ca6-e392-45a0-9514-d370436392ef/caced042-0264-4901-a3a6-78acc82068a3"
+					(reference "R16")
+					(unit 1)
+				)
 			)
 		)
@@
 		(dnp no)
 		(fields_autoplaced yes)
-		(property "Reference" "#PWR014"
+		(property "Reference" "#PWR068"
 			(at 135.89 119.38 0)
 			(effects
@@
 			(project "Open-PLC-Project"
 				(path "/0d177ca6-e392-45a0-9514-d370436392ef/35842953-03b1-4d1a-a0b9-e32cdca1a04c"
-					(reference "#PWR032")
-					(unit 1)
-				)
-				(path "/0d177ca6-e392-45a0-9514-d370436392ef/caced042-0264-4901-a3a6-78acc82068a3"
-					(reference "#PWR014")
+					(reference "#PWR068")
+					(unit 1)
+				)
+				(path "/0d177ca6-e392-45a0-9514-d370436392ef/caced042-0264-4901-a3a6-78acc82068a3"
+					(reference "#PWR062")
 					(unit 1)
 				)
@@
 		(on_board yes)
 		(dnp no)
-		(property "Reference" "R19"
+		(property "Reference" "R28"
 			(at 134.62 90.17 0)
 			(do_not_autoplace yes)
@@
 					(unit 1)
 				)
+				(path "/0d177ca6-e392-45a0-9514-d370436392ef/caced042-0264-4901-a3a6-78acc82068a3"
+					(reference "R24")
+					(unit 1)
+				)
 			)
 		)
@@
 		(on_board yes)
 		(dnp no)
-		(property "Reference" "R17"
+		(property "Reference" "R26"
 			(at 134.62 85.09 0)
 			(do_not_autoplace yes)
@@
 		(dnp no)
 		(fields_autoplaced yes)
-		(property "Reference" "U4"
+		(property "Reference" "U11"
 			(at 146.05 80.01 0)
 			(do_not_autoplace yes)
@@
 			(project "Open-PLC-Project"
 				(path "/0d177ca6-e392-45a0-9514-d370436392ef/35842953-03b1-4d1a-a0b9-e32cdca1a04c"
-					(reference "U4")
+					(reference "U11")
+					(unit 1)
+				)
+				(path "/0d177ca6-e392-45a0-9514-d370436392ef/caced042-0264-4901-a3a6-78acc82068a3"
+					(reference "U10")
 					(unit 1)
 				)
@@
 		(dnp no)
 		(fields_autoplaced yes)
-		(property "Reference" "C17"
+		(property "Reference" "C41"
 			(at 124.46 111.76 0)
 			(do_not_autoplace yes)
@@
 			(project "Open-PLC-Project"
 				(path "/0d177ca6-e392-45a0-9514-d370436392ef/35842953-03b1-4d1a-a0b9-e32cdca1a04c"
-					(reference "C17")
+					(reference "C41")
+					(unit 1)
+				)
+				(path "/0d177ca6-e392-45a0-9514-d370436392ef/caced042-0264-4901-a3a6-78acc82068a3"
+					(reference "C39")
 					(unit 1)
 				)
@@
 		(dnp no)
 		(fields_autoplaced yes)
-		(property "Reference" "#PWR027"
+		(property "Reference" "#PWR072"
 			(at 173.99 81.28 0)
 			(effects
@@
 			(project "Open-PLC-Project"
 				(path "/0d177ca6-e392-45a0-9514-d370436392ef/35842953-03b1-4d1a-a0b9-e32cdca1a04c"
-					(reference "#PWR067")
-					(unit 1)
-				)
-				(path "/0d177ca6-e392-45a0-9514-d370436392ef/caced042-0264-4901-a3a6-78acc82068a3"
-					(reference "#PWR027")
-					(unit 1)
-				)
+					(reference "#PWR072")
+					(unit 1)
+				)
+				(path "/0d177ca6-e392-45a0-9514-d370436392ef/caced042-0264-4901-a3a6-78acc82068a3"
+					(reference "#PWR066")
+					(unit 1)
+				)

Commit message: [Base 회로도 업데이트] - AIN 입력 4개 추가
Other:
- company: (none) -> -
- title: (none) -> Open-PLC-Project
Changed lines of the file:
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@@
 	(generator_version "8.0")
 	(paper "A4")
+	(title_block
+		(title "Open-PLC-Project")
+		(date "2024-12-01")
+		(company "-")
+		(comment 1 "See the file \"LICENSE\" in the main directory of this archive for more details.")
+		(comment 2 "This file is subject to the terms and conditions of the MIT License.")
+		(comment 3 "Copyright (c) 2024 Yoon-Ki Hong")
+	)
 	(junction
 		(at 135.89 106.68)
@@
 		(dnp no)
 		(fields_autoplaced yes)
-		(property "Reference" "#PWR070"
+		(property "Reference" "#PWR079"
 			(at 166.37 109.22 0)
 			(effects
@@
 			(project "Open-PLC-Project"
 				(path "/0d177ca6-e392-45a0-9514-d370436392ef/35842953-03b1-4d1a-a0b9-e32cdca1a04c"
-					(reference "#PWR070")
+					(reference "#PWR079")
 					(unit 1)
 				)
 				(path "/0d177ca6-e392-45a0-9514-d370436392ef/caced042-0264-4901-a3a6-78acc82068a3"
-					(reference "#PWR064")
+					(reference "#PWR073")
 					(unit 1)
 				)
@@
 		(dnp no)
 		(fields_autoplaced yes)
-		(property "Reference" "#PWR067"
+		(property "Reference" "#PWR076"
 			(at 123.19 119.38 0)
 			(effects
@@
 			(project "Open-PLC-Project"
 				(path "/0d177ca6-e392-45a0-9514-d370436392ef/35842953-03b1-4d1a-a0b9-e32cdca1a04c"
-					(reference "#PWR067")
+					(reference "#PWR076")
 					(unit 1)
 				)
 				(path "/0d177ca6-e392-45a0-9514-d370436392ef/caced042-0264-4901-a3a6-78acc82068a3"
-					(reference "#PWR061")
+					(reference "#PWR070")
 					(unit 1)
 				)
@@
 		(dnp no)
 		(fields_autoplaced yes)
-		(property "Reference" "#PWR071"
+		(property "Reference" "#PWR080"
 			(at 173.99 71.374 0)
 			(effects
@@
 			(project "Open-PLC-Project"
 				(path "/0d177ca6-e392-45a0-9514-d370436392ef/35842953-03b1-4d1a-a0b9-e32cdca1a04c"
-					(reference "#PWR071")
+					(reference "#PWR080")
 					(unit 1)
 				)
 				(path "/0d177ca6-e392-45a0-9514-d370436392ef/caced042-0264-4901-a3a6-78acc82068a3"
-					(reference "#PWR065")
+					(reference "#PWR074")
 					(unit 1)
 				)
@@
 		(dnp no)
 		(fields_autoplaced yes)
-		(property "Reference" "#PWR069"
+		(property "Reference" "#PWR078"
 			(at 166.37 78.994 0)
 			(effects
@@
 			(project "Open-PLC-Project"
 				(path "/0d177ca6-e392-45a0-9514-d370436392ef/35842953-03b1-4d1a-a0b9-e32cdca1a04c"
-					(reference "#PWR069")
+					(reference "#PWR078")
 					(unit 1)
 				)
 				(path "/0d177ca6-e392-45a0-9514-d370436392ef/caced042-0264-4901-a3a6-78acc82068a3"
-					(reference "#PWR063")
+					(reference "#PWR072")
 					(unit 1)
 				)
@@
 		(dnp no)
 		(fields_autoplaced yes)
-		(property "Reference" "#PWR068"
+		(property "Reference" "#PWR077"
 			(at 135.89 119.38 0)
 			(effects
@@
 			(project "Open-PLC-Project"
 				(path "/0d177ca6-e392-45a0-9514-d370436392ef/35842953-03b1-4d1a-a0b9-e32cdca1a04c"
-					(reference "#PWR068")
+					(reference "#PWR077")
 					(unit 1)
 				)
 				(path "/0d177ca6-e392-45a0-9514-d370436392ef/caced042-0264-4901-a3a6-78acc82068a3"
-					(reference "#PWR062")
+					(reference "#PWR071")
 					(unit 1)
 				)
@@
 		(dnp no)
 		(fields_autoplaced yes)
-		(property "Reference" "#PWR072"
+		(property "Reference" "#PWR081"
 			(at 173.99 81.28 0)
 			(effects
@@
 			(project "Open-PLC-Project"
 				(path "/0d177ca6-e392-45a0-9514-d370436392ef/35842953-03b1-4d1a-a0b9-e32cdca1a04c"
-					(reference "#PWR072")
+					(reference "#PWR081")
 					(unit 1)
 				)
 				(path "/0d177ca6-e392-45a0-9514-d370436392ef/caced042-0264-4901-a3a6-78acc82068a3"
-					(reference "#PWR066")
-					(unit 1)
-				)
+					(reference "#PWR075")
+					(unit 1)
+				)
